File: RoyalBlue-nRF54L15.kicad_sch (KiCad schematic)
At the start: 30 parts, among them J1 Conn_01x16_Pin, J2 Conn_01x12_Pin, J4 Conn_01x02_MountingPin, J5 Conn_01x04_MountingPin, J6 Conn_01x05_MountingPin, SW1 SW_Push, SW2 SW_Push, U1 BM15x, U4 W25Q16JVUXIQ, Y1 32.768KHz

Commit message: Updated 02/03/25
Parts:
- removed C12: 100nF, Capacitor_SMD:C_0402_1005Metric, symbol Device:C_Small
- removed C13, C14: 300pF, Capacitor_SMD:C_0402_1005Metric, symbol Device:C_Small
- removed C9: 4.7uF, Capacitor_SMD:C_0402_1005Metric, symbol Device:C_Small
- removed D1: LED_Small, LED_SMD:LED_0603_1608Metric, symbol Device:LED_Small
- removed J1: Conn_01x16_Pin, RoyalBlue-nRF54L15-Connector_PinHeader_2.54mm:PinHeader_1x16_P2.54mm_Vertical, symbol Connector:Conn_01x16_Pin
- removed J2: Conn_01x12_Pin, RoyalBlue-nRF54L15-Connector_PinHeader_2.54mm:PinHeader_1x12_P2.54mm_Vertical, symbol Connector:Conn_01x12_Pin
- removed J4: Conn_01x02_MountingPin, Connector_JST:JST_PH_S2B-PH-SM4-TB_1x02-1MP_P2.00mm_Horizontal, symbol Connector_Generic_MountingPin:Conn_01x02_MountingPin
- removed J5: Conn_01x04_MountingPin, Connector_JST:JST_SH_SM04B-SRSS-TB_1x04-1MP_P1.00mm_Horizontal, symbol Connector_Generic_MountingPin:Conn_01x04_MountingPin
- removed J6: Conn_01x05_MountingPin, RoyalBlue-nRF54L15-Connector_FFC-FPC:CONN-SMD_5P-P0.50_HCTL_HC-FPC-05-09-5RLTAG, symbol Connector_Generic_MountingPin:Conn_01x05_MountingPin
- removed R2, R3, R5, R7: 10kR, Resistor_SMD:R_0402_1005Metric, symbol Device:R_Small_US
- removed R6: 470R, Resistor_SMD:R_0402_1005Metric, symbol Device:R_Small_US
- removed SW1, SW2: SW_Push, Button_Switch_SMD:SW_Push_1P1T_NO_Vertical_Wuerth_434133025816, symbol Switch:SW_Push
- removed TP1, TP2, TP3, TP4: TestPoint, TestPoint:TestPoint_Pad_D2.0mm, symbol Connector:TestPoint
- removed U1: BM15x, nordic-lib-kicad-nrf54-modules:BM15x-LGA-45_15.8x10mm, symbol nordic-lib-kicad-nrf54-modules:BM15x
- removed U4: W25Q16JVUXIQ, Package_SON:Winbond_USON-8-1EP_3x2mm_P0.5mm_EP0.2x1.6mm, symbol Memory_Flash:W25Q32JVZP
- removed Y1: 32.768KHz, Crystal:Crystal_SMD_3215-2Pin_3.2x1.5mm, symbol Device:Crystal_Small
Connections:
- no-connect marks 3 -> 0
Other:
- sheet USB renamed Debugger
- added sheet Connectors (sch/Connectors.kicad_sch)
- added sheet nRF54L15 (sch/nRF54L15.kicad_sch)
- sheet Debugger: file USB.kicad_sch -> sch/Debugger.kicad_sch
- sheet Debugger ports: added SWD_TRG{~{RESET}, SWDIO, SWDCLK}, UART_TRG{TX, RX}, USB{VBUS, CC1, CC2}; removed CC1, CC2, TRG_SWDCLK, TRG_SWDIO, TRG_~{RESET}, UART_RX, UART_TX, VBUS_OUT
- sheet nPM1300: file nPM1300.kicad_sch -> sch/nPM1300.kicad_sch
- sheet nPM1300 ports: added ENABLE, NPM1300{SCL, SDA, INT}, USB{VBUS, CC1, CC2}; removed CC1, CC2, GPIO0, GPIO1, SCL_NPM1300, SDA_NPM1300, VBUS_IN
- note removed: "Battery"
- note removed: "Headers"
- note removed: "Qwiic Connector"
- note removed: "USB-C"
- note removed: "nPM1300"
