File: RoyalBlue54L-Feather.kicad_pcb (KiCad board)
At the start: 8 copper layers, 58.4 x 22.9 mm, 69 parts, among them J1 Conn_01x16_Pin, J2 Conn_01x12_Pin, J3 USB_C_Receptacle_USB2.0_16P, J4 Conn_01x02_MountingPin, J5 Conn_01x04_MountingPin, J6 Conn_01x05_MountingPin, J8 Conn_ARM_SWD_TagConnect_TC203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, SW1 SW_Push, SW2 SW_Push, U1 BM15x, U2 nPM1300-QEXX, U3 TPD3E001DRLR, U4 W25Q16JVUXIQ, U5 nRF52833-QDXX, U6 TXB0106RGY, Y1 32.768KHz, Y2 32MHz

Commit message: Added PCBWay logo
Parts:
- added Ref**: Val**, LordsBoards-Symbol:PCBWayLogo, B.Cu at (141.5, 109.9)
Other:
- board text added: "Sponsored by:"
